File: board/backplate.brd (EAGLE design)
At the start: 68.2 x 43.2 mm, 22 parts, among them IC1 MAX7219CNG, IC2 MAX7219CNG, IC3 MAX7219CNG, IC4 MAX7219CNG

Commit message: 4 routed
Parts:
- IC1, IC2, IC3, IC4: device maxim:DIL24-3 -> backplate:DIL24-3
- JP1, JP2: device SparkFun-Connectors:1X05 -> backplate:1X05
Changed lines of the file:
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@@
 <element name="C1" library="TinyTony_ShenzenReady" library_urn="urn:adsk.eagle:library:2159173" package="0805" package3d_urn="urn:adsk.eagle:package:2160663/2" value="10uF" x="24.303" y="36.047" rot="MR270"/>
 <element name="C2" library="TinyTony_ShenzenReady" library_urn="urn:adsk.eagle:library:2159173" package="0805" package3d_urn="urn:adsk.eagle:package:2160663/2" value=".1uF" x="28.032" y="36.075" rot="MR270"/>
-<element name="IC1" library="maxim" library_urn="urn:adsk.eagle:library:269" package="DIL24-3" package3d_urn="urn:adsk.eagle:package:17515/1" value="MAX7219CNG" x="16.51" y="36.83" smashed="yes">
+<element name="IC1" library="backplate" package="DIL24-3" value="MAX7219CNG" x="16.51" y="36.83" smashed="yes">
 <attribute name="MF" value="MAXIM" x="16.51" y="36.83" size="1.778" layer="27" display="off"/>
 <attribute name="MPN" value="MAX7219CNG" x="16.51" y="36.83" size="1.778" layer="27" display="off"/>
-<attribute name="NAME" x="1.2192" y="34.163" size="1.778" layer="25" ratio="10" rot="R90"/>
+<attribute name="NAME" x="7.747" y="38.0492" size="1.778" layer="25" ratio="10" rot="R180"/>
 <attribute name="OC_FARNELL" value="1523914" x="16.51" y="36.83" size="1.778" layer="27" display="off"/>
 <attribute name="OC_NEWARK" value="34C4018" x="16.51" y="36.83" size="1.778" layer="27" display="off"/>
-<attribute name="VALUE" x="3.048" y="35.941" size="1.778" layer="27" ratio="10"/>
+<attribute name="VALUE" x="10.668" y="35.941" size="0.8128" layer="27" ratio="10"/>
 </element>
 <element name="J1" library="backplate" package="2X8" value="" x="7.62" y="24.13"/>
 <element name="R1" library="rcl" library_urn="urn:adsk.eagle:library:334" package="V526-0" package3d_urn="urn:adsk.eagle:package:23590/1" value="33k" x="31.75" y="25.4" smashed="yes" rot="R90">
-<attribute name="NAME" x="28.9635" y="25.436" size="0.8128" layer="25" rot="R270"/>
+<attribute name="NAME" x="28.9635" y="25.436" size="1.016" layer="25" rot="R270"/>
 <attribute name="SPICEPREFIX" value="R" x="31.75" y="25.4" size="1.778" layer="27" rot="R90" display="off"/>
 <attribute name="VALUE" x="33.147" y="24.384" size="0.4064" layer="27" rot="R90"/>
 </element>
-<element name="JP1" library="SparkFun-Connectors" library_urn="urn:adsk.eagle:library:513" package="1X05" package3d_urn="urn:adsk.eagle:package:38104/1" value="" x="2.54" y="15.24" rot="R90"/>
-<element name="JP2" library="SparkFun-Connectors" library_urn="urn:adsk.eagle:library:513" package="1X05" package3d_urn="urn:adsk.eagle:package:38104/1" value="" x="66.04" y="15.24" rot="R90"/>
-<element name="IC2" library="maxim" library_urn="urn:adsk.eagle:library:269" package="DIL24-3" package3d_urn="urn:adsk.eagle:package:17515/1" value="MAX7219CNG" x="50.8" y="36.83" smashed="yes">
+<element name="JP1" library="backplate" package="1X05" value="" x="2.54" y="15.24" rot="R90"/>
+<element name="JP2" library="backplate" package="1X05" value="" x="66.04" y="15.24" rot="R90"/>
+<element name="IC2" library="backplate" package="DIL24-3" value="MAX7219CNG" x="50.8" y="36.83" smashed="yes">
 <attribute name="MF" value="MAXIM" x="50.8" y="59.69" size="1.778" layer="27" display="off"/>
 <attribute name="MPN" value="MAX7219CNG" x="50.8" y="59.69" size="1.778" layer="27" display="off"/>
-<attribute name="NAME" x="35.5092" y="34.163" size="1.778" layer="25" ratio="10" rot="R90"/>
+<attribute name="NAME" x="40.767" y="38.0492" size="1.778" layer="25" ratio="10" rot="R180"/>
 <attribute name="OC_FARNELL" value="1523914" x="50.8" y="59.69" size="1.778" layer="27" display="off"/>
 <attribute name="OC_NEWARK" value="34C4018" x="50.8" y="59.69" size="1.778" layer="27" display="off"/>
-<attribute name="VALUE" x="37.338" y="35.941" size="1.778" layer="27" ratio="10"/>
+<attribute name="VALUE" x="44.958" y="34.671" size="0.8128" layer="27" ratio="10"/>
 </element>
-<element name="R2" library="rcl" library_urn="urn:adsk.eagle:library:334" package="V526-0" package3d_urn="urn:adsk.eagle:package:23590/1" value="33k" x="35.56" y="25.4" rot="R90">
+<element name="R2" library="rcl" library_urn="urn:adsk.eagle:library:334" package="V526-0" package3d_urn="urn:adsk.eagle:package:23590/1" value="33k" x="35.56" y="25.4" smashed="yes" rot="R90">
+<attribute name="NAME" x="33.909" y="22.987" size="1.016" layer="25" ratio="10" rot="R90"/>
 <attribute name="SPICEPREFIX" value="R" x="12.7" y="25.4" size="1.778" layer="27" rot="R90" display="off"/>
+<attribute name="VALUE" x="38.354" y="22.987" size="1.016" layer="27" ratio="10" rot="R90"/>
 </element>
 <element name="C3" library="TinyTony_ShenzenReady" library_urn="urn:adsk.eagle:library:2159173" package="0805" package3d_urn="urn:adsk.eagle:package:2160663/2" value="10uF" x="60.96" y="6.35" rot="MR270"/>
 <element name="C4" library="TinyTony_ShenzenReady" library_urn="urn:adsk.eagle:library:2159173" package="0805" package3d_urn="urn:adsk.eagle:package:2160663/2" value=".1uF" x="55.88" y="6.35" rot="MR270"/>
 <element name="J2" library="backplate" package="2X8" value="" x="41.91" y="24.13"/>
-<element name="IC3" library="maxim" library_urn="urn:adsk.eagle:library:269" package="DIL24-3" package3d_urn="urn:adsk.eagle:package:17515/1" value="MAX7219CNG" x="16.51" y="6.35" smashed="yes">
+<element name="IC3" library="backplate" package="DIL24-3" value="MAX7219CNG" x="16.51" y="6.35" smashed="yes">
 <attribute name="MF" value="MAXIM" x="16.51" y="29.21" size="1.778" layer="27" display="off"/>
 <attribute name="MPN" value="MAX7219CNG" x="16.51" y="29.21" size="1.778" layer="27" display="off"/>
-<attribute name="NAME" x="1.2192" y="3.683" size="1.778" layer="25" ratio="10" rot="R90"/>
+<attribute name="NAME" x="6.477" y="7.5692" size="1.778" layer="25" ratio="10" rot="R180"/>
 <attribute name="OC_FARNELL" value="1523914" x="16.51" y="29.21" size="1.778" layer="27" display="off"/>
 <attribute name="OC_NEWARK" value="34C4018" x="16.51" y="29.21" size="1.778" layer="27" display="off"/>
-<attribute name="VALUE" x="3.048" y="5.461" size="1.778" layer="27" ratio="10"/>
+<attribute name="VALUE" x="4.318" y="4.191" size="0.8128" layer="27" ratio="10"/>
 </element>
-<element name="R3" library="rcl" library_urn="urn:adsk.eagle:library:334" package="V526-0" package3d_urn="urn:adsk.eagle:package:23590/1" value="33k" x="31.75" y="16.51" rot="R90">
+<element name="R3" library="rcl" library_urn="urn:adsk.eagle:library:334" package="V526-0" package3d_urn="urn:adsk.eagle:package:23590/1" value="33k" x="31.75" y="16.51" smashed="yes" rot="R90">
+<attribute name="NAME" x="32.639" y="20.32" size="1.016" layer="25" ratio="10" rot="R180"/>
 <attribute name="SPICEPREFIX" value="R" x="8.89" y="16.51" size="1.778" layer="27" rot="R90" display="off"/>
+<attribute name="VALUE" x="34.544" y="14.097" size="1.016" layer="27" ratio="10" rot="R90"/>
 </element>
 <element name="C5" library="TinyTony_ShenzenReady" library_urn="urn:adsk.eagle:library:2159173" package="0805" package3d_urn="urn:adsk.eagle:package:2160663/2" value="10uF" x="26.67" y="6.35" rot="MR270"/>
 <element name="C6" library="TinyTony_ShenzenReady" library_urn="urn:adsk.eagle:library:2159173" package="0805" package3d_urn="urn:adsk.eagle:package:2160663/2" value=".1uF" x="21.59" y="6.35" rot="MR270"/>
 <element name="J3" library="backplate" package="2X8" value="" x="7.62" y="15.24"/>
-<element name="IC4" library="maxim" library_urn="urn:adsk.eagle:library:269" package="DIL24-3" package3d_urn="urn:adsk.eagle:package:17515/1" value="MAX7219CNG" x="50.8" y="6.35" smashed="yes">
+<element name="IC4" library="backplate" package="DIL24-3" value="MAX7219CNG" x="50.8" y="6.35" smashed="yes">
 <attribute name="MF" value="MAXIM" x="50.8" y="29.21" size="1.778" layer="27" display="off"/>
 <attribute name="MPN" value="MAX7219CNG" x="50.8" y="29.21" size="1.778" layer="27" display="off"/>
-<attribute name="NAME" x="35.5092" y="3.683" size="1.778" layer="25" ratio="10" rot="R90"/>
+<attribute name="NAME" x="40.767" y="7.5692" size="1.778" layer="25" ratio="10" rot="R180"/>
 <attribute name="OC_FARNELL" value="1523914" x="50.8" y="29.21" size="1.778" layer="27" display="off"/>
 <attribute name="OC_NEWARK" value="34C4018" x="50.8" y="29.21" size="1.778" layer="27" display="off"/>
-<attribute name="VALUE" x="37.338" y="5.461" size="1.778" layer="27" ratio="10"/>
+<attribute name="VALUE" x="47.498" y="4.191" size="0.8128" layer="27" ratio="10"/>
 </element>
-<element name="R4" library="rcl" library_urn="urn:adsk.eagle:library:334" package="V526-0" package3d_urn="urn:adsk.eagle:package:23590/1" value="33k" x="35.56" y="16.51" rot="R90">
+<element name="R4" library="rcl" library_urn="urn:adsk.eagle:library:334" package="V526-0" package3d_urn="urn:adsk.eagle:package:23590/1" value="33k" x="35.56" y="16.51" smashed="yes" rot="R90">
+<attribute name="NAME" x="36.957" y="20.32" size="1.016" layer="25" ratio="10" rot="R180"/>
 <attribute name="SPICEPREFIX" value="R" x="12.7" y="16.51" size="1.778" layer="27" rot="R90" display="off"/>
+<attribute name="VALUE" x="38.354" y="14.097" size="1.016" layer="27" ratio="10" rot="R90"/>
 </element>
 <element name="C7" library="TinyTony_ShenzenReady" library_urn="urn:adsk.eagle:library:2159173" package="0805" package3d_urn="urn:adsk.eagle:package:2160663/2" value="10uF" x="58.42" y="36.83" rot="MR90"/>
