File: board/backplate.sch (EAGLE design)
At the start: 7 parts, among them IC1 MAX7219CNG

Commit message: routed 4
Parts:
- added C3, C5, C7: 10uF, TinyTony_ShenzenReady:CAP0805
- added C4, C6, C8: .1uF, TinyTony_ShenzenReady:CAP0805
- added IC2, IC3, IC4: MAX7219CNG, maxim:MAX7219CNG
- added J2, J3, J4: (no value), backplate:CONN_08X2IC
- added R2, R3, R4: 33k, rcl:R-US_V526-0
Connections:
- new net FF: IC1.DOUT, IC2.DIN
- new net N$18: IC2.ISET, R2.2
- new net N$19: IC2.DIG0, J2.8
- new net N$20: IC2.DIG1, J2.5
- new net N$21: IC2.DIG2, J2.7
- new net N$22: IC2.DIG3, J2.14
- new net N$23: IC2.DIG4, J2.11
- new net N$24: IC2.DIG5, J2.12
- new net N$25: IC2.DIG6, J2.4
- new net N$26: IC2.DIG7, J2.2
- new net N$27: IC2.SEGA, J2.6
- new net N$28: IC2.SEGB, J2.15
- new net N$29: IC2.SEGC, J2.10
- new net N$30: IC2.SEGD, J2.1
- new net N$31: IC2.SEGE, J2.13
- new net N$32: IC2.SEGF, J2.3
- new net N$33: IC2.SEGG, J2.9
- new net N$34: IC2.SEGDP, J2.16
- new net N$35: IC3.ISET, R3.2
- new net N$36: IC3.DIG0, J3.8
- new net N$37: IC3.DIG1, J3.5
- new net N$38: IC3.DIG2, J3.7
- new net N$39: IC3.DIG3, J3.14
- new net N$40: IC3.DIG4, J3.11
- new net N$41: IC3.DIG5, J3.12
- new net N$42: IC3.DIG6, J3.4
- new net N$43: IC3.DIG7, J3.2
- new net N$44: IC3.SEGA, J3.6
- new net N$45: IC3.SEGB, J3.15
- new net N$46: IC3.SEGC, J3.10
- new net N$47: IC3.SEGD, J3.1
- new net N$48: IC3.SEGE, J3.13
- new net N$49: IC3.SEGF, J3.3
- new net N$50: IC3.SEGG, J3.9
- new net N$51: IC3.SEGDP, J3.16
- new net N$52: IC4.ISET, R4.2
- new net N$53: IC4.DIG0, J4.8
- new net N$54: IC4.DIG1, J4.5
- new net N$55: IC4.DIG2, J4.7
- new net N$56: IC4.DIG3, J4.14
- new net N$57: IC4.DIG4, J4.11
- new net N$58: IC4.DIG5, J4.12
- new net N$59: IC4.DIG6, J4.4
- new net N$60: IC4.DIG7, J4.2
- new net N$61: IC4.SEGA, J4.6
- new net N$62: IC4.SEGB, J4.15
- new net N$63: IC4.SEGC, J4.10
- new net N$64: IC4.SEGD, J4.1
- new net N$65: IC4.SEGE, J4.13
- new net N$66: IC4.SEGF, J4.3
- new net N$67: IC4.SEGG, J4.9
- new net N$68: IC4.SEGDP, J4.16
- new net N$69: IC2.DOUT, IC4.DIN
- new net N$70: IC3.DIN, IC4.DOUT
- net CLK: now also IC2.CLK, IC3.CLK, IC4.CLK
- net CS: now also IC2.LOAD, IC3.LOAD, IC4.LOAD
- net DOUT: now also IC3.DOUT; no longer IC1.DOUT
- net GND: now also C3.2, C4.2, C5.2, C6.2, C7.2, C8.2, IC2.GND@1, IC2.GND@2, IC3.GND@1, IC3.GND@2, IC4.GND@1, IC4.GND@2
- net VCC: now also C3.1, C4.1, C5.1, C6.1, C7.1, C8.1, IC2.VCC, IC3.VCC, IC4.VCC, R2.1, R3.1, R4.1

Commit message: 4 routed
Parts:
- IC1, IC2, IC3, IC4: device maxim:MAX7219CNG -> backplate:MAX7219CNG
- JP1, JP2: device SparkFun-Connectors:CONN_05 -> backplate:CONN_05
Changed lines of the file:
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@@
 </classes>
 <parts>
-<part name="IC1" library="maxim" library_urn="urn:adsk.eagle:library:269" deviceset="MAX7219CNG" device="" package3d_urn="urn:adsk.eagle:package:17515/1"/>
+<part name="IC1" library="backplate" deviceset="MAX7219CNG" device=""/>
 <part name="R1" library="rcl" library_urn="urn:adsk.eagle:library:334" deviceset="R-US_" device="V526-0" package3d_urn="urn:adsk.eagle:package:23590/1" value="33k"/>
 <part name="P+1" library="supply1" library_urn="urn:adsk.eagle:library:371" deviceset="VCC" device=""/>
@@
 <part name="GND1" library="TinyTony_ShenzenReady" library_urn="urn:adsk.eagle:library:2159173" deviceset="GND" device=""/>
 <part name="J1" library="backplate" deviceset="CONN_08X2" device="IC"/>
-<part name="JP1" library="SparkFun-Connectors" library_urn="urn:adsk.eagle:library:513" deviceset="CONN_05" device="" package3d_urn="urn:adsk.eagle:package:38104/1"/>
-<part name="JP2" library="SparkFun-Connectors" library_urn="urn:adsk.eagle:library:513" deviceset="CONN_05" device="" package3d_urn="urn:adsk.eagle:package:38104/1"/>
-<part name="IC2" library="maxim" library_urn="urn:adsk.eagle:library:269" deviceset="MAX7219CNG" device="" package3d_urn="urn:adsk.eagle:package:17515/1"/>
+<part name="JP1" library="backplate" deviceset="CONN_05" device=""/>
+<part name="JP2" library="backplate" deviceset="CONN_05" device=""/>
+<part name="IC2" library="backplate" deviceset="MAX7219CNG" device=""/>
 <part name="R2" library="rcl" library_urn="urn:adsk.eagle:library:334" deviceset="R-US_" device="V526-0" package3d_urn="urn:adsk.eagle:package:23590/1" value="33k"/>
 <part name="P+3" library="supply1" library_urn="urn:adsk.eagle:library:371" deviceset="VCC" device=""/>
@@
 <part name="GND2" library="TinyTony_ShenzenReady" library_urn="urn:adsk.eagle:library:2159173" deviceset="GND" device=""/>
 <part name="J2" library="backplate" deviceset="CONN_08X2" device="IC"/>
-<part name="IC3" library="maxim" library_urn="urn:adsk.eagle:library:269" deviceset="MAX7219CNG" device="" package3d_urn="urn:adsk.eagle:package:17515/1"/>
+<part name="IC3" library="backplate" deviceset="MAX7219CNG" device=""/>
 <part name="R3" library="rcl" library_urn="urn:adsk.eagle:library:334" deviceset="R-US_" device="V526-0" package3d_urn="urn:adsk.eagle:package:23590/1" value="33k"/>
 <part name="P+5" library="supply1" library_urn="urn:adsk.eagle:library:371" deviceset="VCC" device=""/>
@@
 <part name="GND3" library="TinyTony_ShenzenReady" library_urn="urn:adsk.eagle:library:2159173" deviceset="GND" device=""/>
 <part name="J3" library="backplate" deviceset="CONN_08X2" device="IC"/>
-<part name="IC4" library="maxim" library_urn="urn:adsk.eagle:library:269" deviceset="MAX7219CNG" device="" package3d_urn="urn:adsk.eagle:package:17515/1"/>
+<part name="IC4" library="backplate" deviceset="MAX7219CNG" device=""/>
 <part name="R4" library="rcl" library_urn="urn:adsk.eagle:library:334" deviceset="R-US_" device="V526-0" package3d_urn="urn:adsk.eagle:package:23590/1" value="33k"/>
 <part name="P+7" library="supply1" library_urn="urn:adsk.eagle:library:371" deviceset="VCC" device=""/>
